File: kicad/mppt-2420-hc.kicad_pcb (KiCad board)
At the start: 4 copper layers, 100 x 100 mm, 172 parts, among them J1 MKDS 5/ 2-9,5, J2 MKDS 5/ 2-9,5, J3 MKDS 5/ 2-9,5, J4 8P8C, J5 8P8C, J6 JST PH, J7 UEXT, P1 CONN_01X02, Q1 IPA045N10N3G, Q2 IPA045N10N3G, Q3 IPA045N10N3G, Q4 BUK98180-100A, Q7 IPA045N10N3G, T1 BC846B, T10 BC846B, T2 BC846B, T3 BC846B, T4 BC856B, T5 BC846B, U1 LM5107, U2 STM32G431CBTx, U3 INA186, U4 LMR16006X, U5 INA186, U6 W25Q80DVS, U7 TCAN334, Y1 8MHz

Commit message: Update
Connections:
- net /MCU/~RESET renamed /MCU/~{RESET}
Routing:
- added copper zone on In2.Cu, net +3V3
- added copper zone on In2.Cu, net /DC/DC/SHUNT_DCDC_P
- added copper zone on In1.Cu, net /DC/DC/SW_NODE
- added copper zone on In2.Cu, net /DC/DC/SW_NODE
- added copper zone on In2.Cu, net /DCDC_HV+
- added copper zone on In1.Cu, net GND
- removed copper zone on 3V3, net +3V3
- removed copper zone on 3V3, net /DC/DC/SHUNT_DCDC_P
- removed copper zone on 3V3, net /DC/DC/SW_NODE
- removed copper zone on GND, net /DC/DC/SW_NODE
- removed copper zone on 3V3, net /DCDC_HV+
- removed copper zone on GND, net GND
Other:
- net class Default removed
- net class Power removed
- board text added: "~{RESET}"
- board text removed: "|+S-|"
- board text removed: "~RESET"
